File: eagle/analog/analog.sch (EAGLE design)
At the start: 66 parts, among them IC1 AD8397, IC2 LMV762MA, IC3 AD8632

Commit message: analog
Parts:
- removed C1, C10, C11, C16, C24, C25, C26, C27, C28, C29, C7, C8, C9: (no value), rcl:C-EUC0805
- removed R16, R17, R18, R19, R20, R21, R24, R25, R26, R27, R28, R29, R30: (no value), rcl:R-EU_R0805
- added SV1: (no value), con-lstb:MA03-1
Connections:
- removed net N$12: C21.1, C23.1
- removed net N$15: IC3A.IN-
- removed net N$18: C21.2, C23.2
- removed net N$20: R4.2
- removed net N$22: C13.2, D1.A1
- removed net N$27: C17.2, R22.1
- removed net N$6: L2.2, R6.1, R8.1
- removed net N$9: C15.2, C18.2, C2.2, C22.2, C3.2, L2.1, R10.1, R3.1
- new net +5V: C21.1, C23.1, IC1P.V+, IC2P.V+, IC3P.V+, R23.1
- new net GND: C13.2, C15.2, C17.2, C18.2, C19.1, C2.2, C20.1, C21.2, C22.2, C23.2, C3.2, D1.A1, IC1P.V-, IC2P.V-, IC3P.V-, L2.1, L2.2, R10.1, R22.1, R3.1, R6.1, R8.1, SV1.2
- net N$11: now also SV1.3
- net N$17: now also SV1.1
- net N$30: now also IC3A.IN-
- net N$8: now also R4.2
Other:
- moved on the sheet: C22

Commit message: analog
Parts:
- added U1: MAX4642EUA, analog:MAX4642EUA
Connections:
- new net N$9: IC2B.OUT, U1.IN1
- net +5V: now also U1.V+
- net GND: now also U1.GND
- net N$1: now also U1.IN2
- net N$2: now also U1.COM1, U1.COM2; no longer IC2B.OUT
Other:
- moved on the sheet: C21, C23
Changed lines of the file:
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@@
 <part name="SV1" library="con-lstb" library_urn="urn:adsk.eagle:library:162" deviceset="MA03-1" device="" package3d_urn="urn:adsk.eagle:package:8339/1"/>
 <part name="GND11" library="supply1" library_urn="urn:adsk.eagle:library:371" deviceset="GND" device=""/>
+<part name="U1" library="analog" deviceset="MAX4642EUA" device=""/>
+<part name="GND12" library="supply1" library_urn="urn:adsk.eagle:library:371" deviceset="GND" device=""/>
+<part name="SUPPLY6" library="supply2" library_urn="urn:adsk.eagle:library:372" deviceset="+5V" device=""/>
 </parts>
 <sheets>
@@
 <instance part="C19" gate="G$1" x="175.26" y="83.82" rot="R90"/>
 <instance part="C20" gate="G$1" x="198.12" y="60.96" rot="R90"/>
-<instance part="C21" gate="G$1" x="231.14" y="119.38"/>
+<instance part="C21" gate="G$1" x="182.88" y="160.02"/>
 <instance part="C22" gate="G$1" x="170.18" y="40.64"/>
-<instance part="C23" gate="G$1" x="218.44" y="119.38"/>
+<instance part="C23" gate="G$1" x="170.18" y="160.02"/>
 <instance part="R1" gate="G$1" x="30.48" y="58.42"/>
 <instance part="R2" gate="G$1" x="114.3" y="66.04" rot="R90"/>
@@
 <instance part="SUPPLY3" gate="+5V" x="157.48" y="160.02"/>
 <instance part="GND7" gate="1" x="119.38" y="96.52" rot="R90"/>
-<instance part="GND8" gate="1" x="246.38" y="111.76"/>
+<instance part="GND8" gate="1" x="198.12" y="152.4"/>
 <instance part="GND9" gate="1" x="172.72" y="114.3"/>
-<instance part="SUPPLY4" gate="+5V" x="246.38" y="124.46"/>
+<instance part="SUPPLY4" gate="+5V" x="198.12" y="165.1"/>
 <instance part="SUPPLY5" gate="+5V" x="172.72" y="137.16"/>
 <instance part="GND10" gate="1" x="12.7" y="30.48"/>
 <instance part="SV1" gate="G$1" x="12.7" y="81.28"/>
 <instance part="GND11" gate="1" x="22.86" y="81.28" rot="R90"/>
+<instance part="U1" gate="A" x="203.2" y="144.78"/>
+<instance part="GND12" gate="1" x="205.74" y="132.08"/>
+<instance part="SUPPLY6" gate="+5V" x="243.84" y="149.86"/>
 </instances>
 <busses>
 </busses>
 <nets>
-<net name="N$1" class="0">
-<segment>
-<pinref part="IC2" gate="A" pin="OUT"/>
-<wire x1="233.68" y1="81.28" x2="243.84" y2="81.28" width="0.1524" layer="91"/>
-</segment>
-</net>
-<net name="N$2" class="0">
-<segment>
-<pinref part="IC2" gate="B" pin="OUT"/>
-<wire x1="233.68" y1="63.5" x2="243.84" y2="63.5" width="0.1524" layer="91"/>
-</segment>
-</net>
 <net name="N$3" class="0">
 <segment>
@@
 <pinref part="GND8" gate="1" pin="GND"/>
 <pinref part="C21" gate="G$1" pin="2"/>
-<wire x1="246.38" y1="114.3" x2="231.14" y2="114.3" width="0.1524" layer="91"/>
+<wire x1="198.12" y1="154.94" x2="182.88" y2="154.94" width="0.1524" layer="91"/>
 <pinref part="C23" gate="G$1" pin="2"/>
-<wire x1="218.44" y1="114.3" x2="231.14" y2="114.3" width="0.1524" layer="91"/>
-<junction x="231.14" y="114.3"/>
+<wire x1="170.18" y1="154.94" x2="182.88" y2="154.94" width="0.1524" layer="91"/>
+<junction x="182.88" y="154.94"/>
 </segment>
 <segment>
@@
 <pinref part="GND11" gate="1" pin="GND"/>
 </segment>
+<segment>
+<pinref part="U1" gate="A" pin="GND"/>
+<pinref part="GND12" gate="1" pin="GND"/>
+<wire x1="205.74" y1="137.16" x2="205.74" y2="134.62" width="0.1524" layer="91"/>
+</segment>
 </net>
 <net name="+5V" class="0">
@@
 <pinref part="SUPPLY4" gate="+5V" pin="+5V"/>
 <pinref part="C21" gate="G$1" pin="1"/>
-<wire x1="246.38" y1="121.92" x2="231.14" y2="121.92" width="0.1524" layer="91"/>
+<wire x1="198.12" y1="162.56" x2="182.88" y2="162.56" width="0.1524" layer="91"/>
 <pinref part="C23" gate="G$1" pin="1"/>
-<wire x1="218.44" y1="121.92" x2="231.14" y2="121.92" width="0.1524" layer="91"/>
-<junction x="231.14" y="121.92"/>
+<wire x1="170.18" y1="162.56" x2="182.88" y2="162.56" width="0.1524" layer="91"/>
+<junction x="182.88" y="162.56"/>
 </segment>
 <segment>
@@
 <wire x1="172.72" y1="134.62" x2="175.26" y2="134.62" width="0.1524" layer="91"/>
 </segment>
-</net>
+<segment>
+<pinref part="U1" gate="A" pin="V+"/>
+<wire x1="241.3" y1="144.78" x2="243.84" y2="144.78" width="0.1524" layer="91"/>
+<pinref part="SUPPLY6" gate="+5V" pin="+5V"/>
+<wire x1="243.84" y1="144.78" x2="243.84" y2="147.32" width="0.1524" layer="91"/>
+</segment>
+</net>
+<net name="N$1" class="0">
+<segment>
+<pinref part="IC2" gate="A" pin="OUT"/>
+<pinref part="U1" gate="A" pin="IN2"/>
+<wire x1="233.68" y1="81.28" x2="233.68" y2="114.3" width="0.1524" layer="91"/>
+<wire x1="233.68" y1="114.3" x2="233.68" y2="121.92" width="0.1524" layer="91"/>
+<wire x1="233.68" y1="121.92" x2="203.2" y2="121.92" width="0.1524" layer="91"/>
+<wire x1="203.2" y1="121.92" x2="203.2" y2="139.7" width="0.1524" layer="91"/>
+<wire x1="203.2" y1="139.7" x2="205.74" y2="139.7" width="0.1524" layer="91"/>
+</segment>
+</net>
+<net name="N$2" class="0">
+<segment>
+<pinref part="U1" gate="A" pin="COM1"/>
+<wire x1="205.74" y1="142.24" x2="200.66" y2="142.24" width="0.1524" layer="91"/>
+<wire x1="200.66" y1="142.24" x2="200.66" y2="127" width="0.1524" layer="91"/>
+<wire x1="200.66" y1="127" x2="251.46" y2="127" width="0.1524" layer="91"/>
+<wire x1="251.46" y1="127" x2="251.46" y2="139.7" width="0.1524" layer="91"/>
+<pinref part="U1" gate="A" pin="COM2"/>
+<wire x1="251.46" y1="139.7" x2="241.3" y2="139.7" width="0.1524" layer="91"/>
+</segment>
+</net>
+<net name="N$9" class="0">
+<segment>
+<pinref part="U1" gate="A" pin="IN1"/>
+<wire x1="246.38" y1="142.24" x2="241.3" y2="142.24" width="0.1524" layer="91"/>
+<wire x1="246.38" y1="63.5" x2="246.38" y2="142.24" width="0.1524" layer="91"/>
+<pinref part="IC2" gate="B" pin="OUT"/>
+<wire x1="233.68" y1="63.5" x2="246.38" y2="63.5" width="0.1524" layer="91"/>
+</segment>
+</net>
