File: kicad/analog.sch (KiCad schematic (older format))
At the start: 9 parts

Commit message: schematic
Parts:
- added C?: C, symbol C
- added L?: Ferrite_Bead, symbol Ferrite_Bead
Connections:
- net at U?.2 (-), U?.5 (+): no longer R?.1
- net at U?.3 (+): now also R?.1, R?.2
- net at R?.1, R?.2, U?.6 (-): now also C?.1
- net GNDD: now reaches R?.2
- net GNDD: now also R?.2, C?.2, L?.1
- net at R?.1: now also R?.1
Other:
- moved on the sheet: R?
Changed lines of the file:
@@
 LIBS:contrib
 LIBS:valves
+LIBS:analog-cache
 EELAYER 25 0
 EELAYER END
@@
 L R R?
 U 1 1 5A3ABAB9
-P 8200 4800
-F 0 "R?" V 8280 4800 50  0000 C CNN
-F 1 "R" V 8200 4800 50  0000 C CNN
-F 2 "" V 8130 4800 50  0001 C CNN
-F 3 "" H 8200 4800 50  0001 C CNN
-	1    8200 4800
+P 7800 4800
+F 0 "R?" V 7880 4800 50  0000 C CNN
+F 1 "R" V 7800 4800 50  0000 C CNN
+F 2 "" V 7730 4800 50  0001 C CNN
+F 3 "" H 7800 4800 50  0001 C CNN
+	1    7800 4800
 	1    0    0    -1
 $EndComp
@@
 L R R?
 U 1 1 5A3ABB00
-P 8200 3600
-F 0 "R?" V 8280 3600 50  0000 C CNN
-F 1 "R" V 8200 3600 50  0000 C CNN
-F 2 "" V 8130 3600 50  0001 C CNN
-F 3 "" H 8200 3600 50  0001 C CNN
-	1    8200 3600
+P 7800 3600
+F 0 "R?" V 7880 3600 50  0000 C CNN
+F 1 "R" V 7800 3600 50  0000 C CNN
+F 2 "" V 7730 3600 50  0001 C CNN
+F 3 "" H 7800 3600 50  0001 C CNN
+	1    7800 3600
 	1    0    0    -1
 $EndComp
+$Comp
+L C C?
+U 1 1 5A3AC10E
+P 8700 5450
+F 0 "C?" H 8725 5550 50  0000 L CNN
+F 1 "C" H 8725 5350 50  0000 L CNN
+F 2 "" H 8738 5300 50  0001 C CNN
+F 3 "" H 8700 5450 50  0001 C CNN
+	1    8700 5450
+	0    1    1    0
+$EndComp
+$Comp
+L GNDD #PWR?
+U 1 1 5A3AC6C9
+P 8300 5450
+F 0 "#PWR?" H 8300 5200 50  0001 C CNN
+F 1 "GNDD" H 8300 5325 50  0000 C CNN
+F 2 "" H 8300 5450 50  0001 C CNN
+F 3 "" H 8300 5450 50  0001 C CNN
+	1    8300 5450
+	0    1    1    0
+$EndComp
+$Comp
+L GNDD #PWR?
+U 1 1 5A3ACCB5
+P 9900 6300
+F 0 "#PWR?" H 9900 6050 50  0001 C CNN
+F 1 "GNDD" H 9900 6175 50  0000 C CNN
+F 2 "" H 9900 6300 50  0001 C CNN
+F 3 "" H 9900 6300 50  0001 C CNN
+	1    9900 6300
+	0    -1   -1   0
+$EndComp
+$Comp
+L Ferrite_Bead L?
+U 1 1 5A3ACFE4
+P 7350 6300
+F 0 "L?" V 7200 6325 50  0000 C CNN
+F 1 "Ferrite_Bead" V 7500 6300 50  0000 C CNN
+F 2 "" V 7280 6300 50  0001 C CNN
+F 3 "" H 7350 6300 50  0001 C CNN
+	1    7350 6300
+	0    1    1    0
+$EndComp
 Wire Wire Line
-	9500 5450 9150 5450
+	8850 5450 9500 5450
 Wire Wire Line
 	9150 4950 9150 5800
 Connection ~ 9150 5450
 Wire Wire Line
-	9500 4300 9150 4300
+	8300 5450 8550 5450
 Wire Wire Line
-	9150 4300 9150 4650
+	7500 6300 9900 6300
+Wire Wire Line
+	9150 6300 9150 6100
+Wire Wire Line
+	7800 6300 7800 4950
+Connection ~ 9150 6300
+Connection ~ 7800 6300
 Wire Wire Line
 	9500 5250 9350 5250
 Wire Wire Line
 	9350 5250 9350 4300
-Connection ~ 9350 4300
+Wire Wire Line
+	9350 4300 9500 4300
+Wire Wire Line
+	9500 4100 7800 4100
+Wire Wire Line
+	7800 3750 7800 4650
+Connection ~ 7800 4100
+Wire Wire Line
+	9150 4650 9150 3200
+Wire Wire Line
+	9150 3200 7800 3200
+Wire Wire Line
+	7800 3200 7800 3450
 $EndSCHEMATC

Commit message: pokazhi
Parts:
- added C? (x8): C, symbol C
- added L?: Ferrite_Bead, symbol Ferrite_Bead
- added L?: L_Core_Ferrite, symbol L_Core_Ferrite
- added R? (x7): R, symbol R
Connections:
- net GNDD: now also C?.2, C?.2, R?.2
- net at U?.1: now also L?.2, R?.2
- net at U?.2 (-): now also R?.1, R?.2
- net at R?.1, R?.2, U?.3 (+): now also C?.1
- net at U?.1: now also R?.1, R?.1, C?.1, L?.1
- net at U?.2 (-): now also C?.1, R?.1, R?.1
- net at U?.3 (+): now also R?.2
- net at L?.2: now also C?.2, C?.2, R?.2, R?.2
- new net: C?.1, C?.1, L?.2, R?.1
- new net: C?.2, R?.1
- new net: C?.2, C?.2, C?.2, R?.1
- new net: C?.1, C?.1, C?.1, L?.1
- new net +5V: R?.2
Other:
- moved on the sheet: C?, L?, R?, U?A

Commit message: schematic
Parts:
- added C? (x4): C, symbol C
- added R? (x2): R, symbol R
Connections:
- net GNDD: now also C?.2, C?.2, L?.2, R?.2, R?.2, C?.2, C?.2, C?.2, C?.2
- net at R?.1, R?.2, U?.2 (-): now also C?.1
- net at U?.3 (+): now also C?.1, R?.1
- net at R?.2, U?.3 (+): now also R?.1
- net at R?.1: now also C?.1, R?.2
- new net: C?.1, R?.2
Other:
- moved on the sheet: C?, L?, R?, U?A, U?B

Commit message: lil
Parts:
- added D?: D_Schottky_x2_Serial_AKC, symbol D_Schottky_x2_Serial_AKC
Changed lines of the file:
@@
 	5400 4050 1500 4050
 Connection ~ 1500 4900
+$Comp
+L D_Schottky_x2_Serial_AKC D?
+U 1 1 5A3C3423
+P 4350 2700
+F 0 "D?" H 4400 2600 50  0000 C CNN
+F 1 "D_Schottky_x2_Serial_AKC" H 4350 2800 50  0000 C CNN
+F 2 "" H 4350 2700 50  0001 C CNN
+F 3 "" H 4350 2700 50  0001 C CNN
+	1    4350 2700
+	1    0    0    -1
+$EndComp
 $EndSCHEMATC

Commit message: pochemu
Parts:
- added C?: C, symbol C
- added R? (x3): R, symbol R
Connections:
- net GNDD: now also D?.2 (K)
- net at C?.1, R?.1, R?.2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: now also R?.2
- net at C?.1, R?.1, U?.3 (+): now also R?.2
- net at U?.5 (+): now also R?.1, R?.2
- net at U?.6 (-): now also R?.1
- net at U?.7: now also C?.1, R?.1
- net at C?.1, R?.2: now also D?.1 (A)
- net at D?.3 (common): now also C?.2
Other:
- moved on the sheet: D?, U?B

Commit message: sim
Parts:
- added J?: Conn_01x03, symbol Conn_01x03
- added R?: R, symbol R
Connections:
- net GNDD: now also J?.2 (Pin_2); no longer C?.2, C?.2, C?.2, C?.2, C?.2, L?.2, R?.2, R?.2
- net at C?.1, R?.1, R?.2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: now also J?.1 (Pin_1), R?.2
- net at U?.2 (-), U?.5 (+): now also R?.1
- net at C?.1, L?.2: no longer C?.1, R?.1
- net at C?.1, C?.1, C?.1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: now also J?.3 (Pin_3)
- new net: C?.1, R?.1
- new net GNDPWR: C?.2, C?.2, C?.2, C?.2, C?.2, L?.2, R?.2, R?.2
Other:
- moved on the sheet: R?
