File: eagle/zxclone/board.sch (EAGLE design)
At the start: 0 parts

Commit message: z80
Parts:
- added IC1: (no value), zilog:Z80CPU
Changed lines of the file:
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@@
 <grid distance="0.1" unitdist="inch" unit="inch" style="lines" multiple="1" display="no" altdistance="0.01" altunitdist="inch" altunit="inch"/>
 <layers>
+<layer number="1" name="Top" color="4" fill="1" visible="no" active="no"/>
+<layer number="16" name="Bottom" color="1" fill="1" visible="no" active="no"/>
+<layer number="17" name="Pads" color="2" fill="1" visible="no" active="no"/>
+<layer number="18" name="Vias" color="2" fill="1" visible="no" active="no"/>
+<layer number="19" name="Unrouted" color="6" fill="1" visible="no" active="no"/>
+<layer number="20" name="Dimension" color="15" fill="1" visible="no" active="no"/>
+<layer number="21" name="tPlace" color="7" fill="1" visible="no" active="no"/>
+<layer number="22" name="bPlace" color="7" fill="1" visible="no" active="no"/>
+<layer number="23" name="tOrigins" color="15" fill="1" visible="no" active="no"/>
+<layer number="24" name="bOrigins" color="15" fill="1" visible="no" active="no"/>
+<layer number="25" name="tNames" color="7" fill="1" visible="no" active="no"/>
+<layer number="26" name="bNames" color="7" fill="1" visible="no" active="no"/>
+<layer number="27" name="tValues" color="7" fill="1" visible="no" active="no"/>
+<layer number="28" name="bValues" color="7" fill="1" visible="no" active="no"/>
+<layer number="29" name="tStop" color="7" fill="3" visible="no" active="no"/>
+<layer number="30" name="bStop" color="7" fill="6" visible="no" active="no"/>
+<layer number="31" name="tCream" color="7" fill="4" visible="no" active="no"/>
+<layer number="32" name="bCream" color="7" fill="5" visible="no" active="no"/>
+<layer number="33" name="tFinish" color="6" fill="3" visible="no" active="no"/>
+<layer number="34" name="bFinish" color="6" fill="6" visible="no" active="no"/>
+<layer number="35" name="tGlue" color="7" fill="4" visible="no" active="no"/>
+<layer number="36" name="bGlue" color="7" fill="5" visible="no" active="no"/>
+<layer number="37" name="tTest" color="7" fill="1" visible="no" active="no"/>
+<layer number="38" name="bTest" color="7" fill="1" visible="no" active="no"/>
+<layer number="39" name="tKeepout" color="4" fill="11" visible="no" active="no"/>
+<layer number="40" name="bKeepout" color="1" fill="11" visible="no" active="no"/>
+<layer number="41" name="tRestrict" color="4" fill="10" visible="no" active="no"/>
+<layer number="42" name="bRestrict" color="1" fill="10" visible="no" active="no"/>
+<layer number="43" name="vRestrict" color="2" fill="10" visible="no" active="no"/>
+<layer number="44" name="Drills" color="7" fill="1" visible="no" active="no"/>
+<layer number="45" name="Holes" color="7" fill="1" visible="no" active="no"/>
+<layer number="46" name="Milling" color="3" fill="1" visible="no" active="no"/>
+<layer number="47" name="Measures" color="7" fill="1" visible="no" active="no"/>
+<layer number="48" name="Document" color="7" fill="1" visible="no" active="no"/>
+<layer number="49" name="Reference" color="7" fill="1" visible="no" active="no"/>
+<layer number="51" name="tDocu" color="7" fill="1" visible="no" active="no"/>
+<layer number="52" name="bDocu" color="7" fill="1" visible="no" active="no"/>
 <layer number="88" name="SimResults" color="9" fill="1" visible="yes" active="yes"/>
 <layer number="89" name="SimProbes" color="9" fill="1" visible="yes" active="yes"/>
@@
 </classes>
 <parts>
+<part name="IC1" library="zilog" library_urn="urn:adsk.eagle:library:419" deviceset="Z80CPU" device="" package3d_urn="urn:adsk.eagle:package:31068/1"/>
 </parts>
 <sheets>
@@
 </plain>
 <instances>
+<instance part="IC1" gate="1" x="76.2" y="45.72"/>
 </instances>
 <busses>
@@
 </schematic>
 </drawing>
+<compatibility>
+<note version="8.2" severity="warning">
+Since Version 8.2, EAGLE supports online libraries. The ids
+of those online libraries will not be understood (or retained)
+with this version.
+</note>
+<note version="8.3" severity="warning">
+Since Version 8.3, EAGLE supports URNs for individual library
+assets (packages, symbols, and devices). The URNs of those assets
+will not be understood (or retained) with this version.
+</note>
+<note version="8.3" severity="warning">
+Since Version 8.3, EAGLE supports the association of 3D packages
+with devices in libraries, schematics, and board files. Those 3D
+packages will not be understood (or retained) with this version.
+</note>
+</compatibility>
 </eagle>

Commit message: SN74LS86
Parts:
- added IC2: 74LS86N, 74xx-us:74LS86N
Connections:
- new net N$1: IC1.CLK, IC2B.O
Changed lines of the file:
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@@
 <parts>
 <part name="IC1" library="zilog" library_urn="urn:adsk.eagle:library:419" deviceset="Z80CPU" device="" package3d_urn="urn:adsk.eagle:package:31068/1"/>
+<part name="IC2" library="74xx-us" library_urn="urn:adsk.eagle:library:88" deviceset="74*86" device="N" package3d_urn="urn:adsk.eagle:package:2921/1" technology="LS"/>
 </parts>
 <sheets>
@@
 <instances>
 <instance part="IC1" gate="1" x="76.2" y="45.72"/>
+<instance part="IC2" gate="A" x="0" y="83.82"/>
+<instance part="IC2" gate="B" x="0" y="66.04"/>
+<instance part="IC2" gate="C" x="0" y="48.26"/>
+<instance part="IC2" gate="D" x="0" y="30.48"/>
 </instances>
 <busses>
 </busses>
 <nets>
+<net name="N$1" class="0">
+<segment>
+<pinref part="IC2" gate="B" pin="O"/>
+<wire x1="12.7" y1="66.04" x2="33.02" y2="66.04" width="0.1524" layer="91"/>
+<wire x1="33.02" y1="66.04" x2="33.02" y2="22.86" width="0.1524" layer="91"/>
+<pinref part="IC1" gate="1" pin="CLK"/>
+<wire x1="33.02" y1="22.86" x2="58.42" y2="22.86" width="0.1524" layer="91"/>
+</segment>
+</net>
 </nets>
 </sheet>

Commit message: board
Connections:
- new net /RAS: IC2A.I0
- new net N$2: IC2A.I1, IC2B.I1
- new net N$3: IC2A.O, IC2B.I0
Other:
- moved on the sheet: IC2A
Changed lines of the file:
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@@
 <instances>
 <instance part="IC1" gate="1" x="76.2" y="45.72"/>
-<instance part="IC2" gate="A" x="0" y="83.82"/>
+<instance part="IC2" gate="A" x="0" y="86.36"/>
 <instance part="IC2" gate="B" x="0" y="66.04"/>
 <instance part="IC2" gate="C" x="0" y="48.26"/>
@@
 </segment>
 </net>
+<net name="N$2" class="0">
+<segment>
+<pinref part="IC2" gate="A" pin="I1"/>
+<wire x1="-12.7" y1="83.82" x2="-20.32" y2="83.82" width="0.1524" layer="91"/>
+<wire x1="-20.32" y1="83.82" x2="-20.32" y2="63.5" width="0.1524" layer="91"/>
+<pinref part="IC2" gate="B" pin="I1"/>
+<wire x1="-20.32" y1="63.5" x2="-12.7" y2="63.5" width="0.1524" layer="91"/>
+</segment>
+</net>
+<net name="N$3" class="0">
+<segment>
+<pinref part="IC2" gate="A" pin="O"/>
+<wire x1="12.7" y1="86.36" x2="17.78" y2="86.36" width="0.1524" layer="91"/>
+<wire x1="17.78" y1="86.36" x2="17.78" y2="76.2" width="0.1524" layer="91"/>
+<wire x1="17.78" y1="76.2" x2="-15.24" y2="76.2" width="0.1524" layer="91"/>
+<wire x1="-15.24" y1="76.2" x2="-15.24" y2="68.58" width="0.1524" layer="91"/>
+<pinref part="IC2" gate="B" pin="I0"/>
+<wire x1="-15.24" y1="68.58" x2="-12.7" y2="68.58" width="0.1524" layer="91"/>
+</segment>
+</net>
+<net name="/RAS" class="0">
+<segment>
+<pinref part="IC2" gate="A" pin="I0"/>
+<wire x1="-12.7" y1="88.9" x2="-71.12" y2="88.9" width="0.1524" layer="91"/>
+<label x="-66.04" y="88.9" size="1.778" layer="95"/>
+</segment>
+</net>

Commit message: board
Parts:
- added IC3: 74LS74N, 74xx-us:74LS74N
- added IC4: 74LS04N, 74xx-us:74LS04N
- added Q1: (no value), crystal:CRYSTALHC49S
- added R1: (no value), resistor:R-US_0207/10
Connections:
- new net N$4: IC3A.!Q, IC3A.D
- new net N$5: IC3A.Q, IC3B.CLK
- new net N$6: IC3A.CLK, IC4B.O, Q1.2
- new net N$7: IC4B.I, IC4C.O, R1.1
- new net N$8: IC4C.I, Q1.1, R1.2
- net /RAS: now also IC3B.Q
Changed lines of the file:
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@@
 <layer number="97" name="Info" color="7" fill="1" visible="yes" active="yes"/>
 <layer number="98" name="Guide" color="6" fill="1" visible="yes" active="yes"/>
+<layer number="99" name="SpiceOrder" color="5" fill="1" visible="yes" active="yes"/>
 </layers>
 <schematic xreflabel="%F%N/%S.%C%R" xrefpart="/%S.%C%R">
@@
 <part name="IC1" library="zilog" library_urn="urn:adsk.eagle:library:419" deviceset="Z80CPU" device="" package3d_urn="urn:adsk.eagle:package:31068/1"/>
 <part name="IC2" library="74xx-us" library_urn="urn:adsk.eagle:library:88" deviceset="74*86" device="N" package3d_urn="urn:adsk.eagle:package:2921/1" technology="LS"/>
+<part name="IC3" library="74xx-us" library_urn="urn:adsk.eagle:library:88" deviceset="74*74" device="N" package3d_urn="urn:adsk.eagle:package:2921/1" technology="LS"/>
+<part name="IC4" library="74xx-us" library_urn="urn:adsk.eagle:library:88" deviceset="74*04" device="N" package3d_urn="urn:adsk.eagle:package:2921/1" technology="LS"/>
+<part name="R1" library="resistor" library_urn="urn:adsk.eagle:library:348" deviceset="R-US_" device="0207/10" package3d_urn="urn:adsk.eagle:package:25939/1"/>
+<part name="Q1" library="crystal" library_urn="urn:adsk.eagle:library:204" deviceset="CRYSTAL" device="HC49S" package3d_urn="urn:adsk.eagle:package:12071/1"/>
 </parts>
 <sheets>
@@
 <instance part="IC2" gate="C" x="0" y="48.26"/>
 <instance part="IC2" gate="D" x="0" y="30.48"/>
+<instance part="IC3" gate="A" x="-81.28" y="88.9"/>
+<instance part="IC3" gate="B" x="-81.28" y="58.42"/>
+<instance part="IC4" gate="A" x="-154.94" y="93.98"/>
+<instance part="IC4" gate="B" x="-154.94" y="73.66"/>
+<instance part="IC4" gate="C" x="-154.94" y="53.34"/>
+<instance part="IC4" gate="D" x="-154.94" y="33.02"/>
+<instance part="IC4" gate="E" x="-154.94" y="15.24"/>
+<instance part="IC4" gate="F" x="-154.94" y="-5.08"/>
+<instance part="R1" gate="G$1" x="-187.96" y="53.34"/>
+<instance part="Q1" gate="G$1" x="-127" y="58.42" rot="R90"/>
 </instances>
 <busses>
@@
 <segment>
 <pinref part="IC2" gate="A" pin="I0"/>
-<wire x1="-12.7" y1="88.9" x2="-71.12" y2="88.9" width="0.1524" layer="91"/>
-<label x="-66.04" y="88.9" size="1.778" layer="95"/>
+<wire x1="-12.7" y1="88.9" x2="-55.88" y2="88.9" width="0.1524" layer="91"/>
+<label x="-53.34" y="88.9" size="1.778" layer="95"/>
+<pinref part="IC3" gate="B" pin="Q"/>
+<wire x1="-55.88" y1="88.9" x2="-55.88" y2="63.5" width="0.1524" layer="91"/>
+<wire x1="-55.88" y1="63.5" x2="-68.58" y2="63.5" width="0.1524" layer="91"/>
 </segment>
 </net>
+<net name="N$4" class="0">
+<segment>
+<pinref part="IC3" gate="A" pin="D"/>
+<wire x1="-93.98" y1="91.44" x2="-96.52" y2="91.44" width="0.1524" layer="91"/>
+<wire x1="-96.52" y1="91.44" x2="-96.52" y2="76.2" width="0.1524" layer="91"/>
+<wire x1="-96.52" y1="76.2" x2="-66.04" y2="76.2" width="0.1524" layer="91"/>
+<wire x1="-66.04" y1="76.2" x2="-66.04" y2="83.82" width="0.1524" layer="91"/>
+<pinref part="IC3" gate="A" pin="!Q"/>
+<wire x1="-66.04" y1="83.82" x2="-68.58" y2="83.82" width="0.1524" layer="91"/>
+</segment>
+</net>
+<net name="N$5" class="0">
+<segment>
+<pinref part="IC3" gate="B" pin="CLK"/>
+<wire x1="-93.98" y1="55.88" x2="-99.06" y2="55.88" width="0.1524" layer="91"/>
+<wire x1="-99.06" y1="55.88" x2="-99.06" y2="71.12" width="0.1524" layer="91"/>
+<wire x1="-99.06" y1="71.12" x2="-63.5" y2="71.12" width="0.1524" layer="91"/>
+<wire x1="-63.5" y1="71.12" x2="-63.5" y2="93.98" width="0.1524" layer="91"/>
+<pinref part="IC3" gate="A" pin="Q"/>
+<wire x1="-63.5" y1="93.98" x2="-68.58" y2="93.98" width="0.1524" layer="91"/>
+</segment>
+</net>
+<net name="N$6" class="0">
+<segment>
+<pinref part="IC3" gate="A" pin="CLK"/>
+<wire x1="-93.98" y1="86.36" x2="-119.38" y2="86.36" width="0.1524" layer="91"/>
+<wire x1="-119.38" y1="86.36" x2="-119.38" y2="73.66" width="0.1524" layer="91"/>
+<pinref part="IC4" gate="B" pin="O"/>
+<wire x1="-119.38" y1="73.66" x2="-127" y2="73.66" width="0.1524" layer="91"/>
+<junction x="-127" y="73.66"/>
+<wire x1="-127" y1="73.66" x2="-144.78" y2="73.66" width="0.1524" layer="91"/>
+<wire x1="-127" y1="73.66" x2="-127" y2="60.96" width="0.1524" layer="91"/>
+<pinref part="Q1" gate="G$1" pin="2"/>
+</segment>
+</net>
+<net name="N$7" class="0">
+<segment>
+<pinref part="IC4" gate="B" pin="I"/>
+<wire x1="-165.1" y1="73.66" x2="-172.72" y2="73.66" width="0.1524" layer="91"/>
+<wire x1="-172.72" y1="73.66" x2="-172.72" y2="68.58" width="0.1524" layer="91"/>
+<wire x1="-172.72" y1="68.58" x2="-172.72" y2="63.5" width="0.1524" layer="91"/>
+<wire x1="-172.72" y1="63.5" x2="-137.16" y2="63.5" width="0.1524" layer="91"/>
+<pinref part="IC4" gate="C" pin="O"/>
+<wire x1="-137.16" y1="63.5" x2="-137.16" y2="53.34" width="0.1524" layer="91"/>
+<wire x1="-137.16" y1="53.34" x2="-144.78" y2="53.34" width="0.1524" layer="91"/>
+<pinref part="R1" gate="G$1" pin="1"/>
+<wire x1="-193.04" y1="53.34" x2="-200.66" y2="53.34" width="0.1524" layer="91"/>
+<wire x1="-200.66" y1="53.34" x2="-200.66" y2="68.58" width="0.1524" layer="91"/>
+<wire x1="-200.66" y1="68.58" x2="-172.72" y2="68.58" width="0.1524" layer="91"/>
+<junction x="-172.72" y="68.58"/>
+</segment>
+</net>
+<net name="N$8" class="0">
+<segment>
+<pinref part="IC4" gate="C" pin="I"/>
+<wire x1="-165.1" y1="53.34" x2="-172.72" y2="53.34" width="0.1524" layer="91"/>
+<pinref part="R1" gate="G$1" pin="2"/>
+<junction x="-172.72" y="53.34"/>
+<wire x1="-172.72" y1="53.34" x2="-182.88" y2="53.34" width="0.1524" layer="91"/>
+<wire x1="-172.72" y1="53.34" x2="-172.72" y2="43.18" width="0.1524" layer="91"/>
+<wire x1="-172.72" y1="43.18" x2="-127" y2="43.18" width="0.1524" layer="91"/>
+<wire x1="-127" y1="43.18" x2="-127" y2="55.88" width="0.1524" layer="91"/>
+<pinref part="Q1" gate="G$1" pin="1"/>
+</segment>
+</net>

Commit message: memory
Parts:
- added IC10, IC11, IC12, IC5, IC6, IC7, IC8, IC9: (no value), memory:2164
Connections:
- net /RAS: now also IC10.!RAS, IC11.!RAS, IC12.!RAS, IC5.!RAS, IC6.!RAS, IC7.!RAS, IC8.!RAS, IC9.!RAS
Changed lines of the file:
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@@
 <part name="R1" library="resistor" library_urn="urn:adsk.eagle:library:348" deviceset="R-US_" device="0207/10" package3d_urn="urn:adsk.eagle:package:25939/1"/>
 <part name="Q1" library="crystal" library_urn="urn:adsk.eagle:library:204" deviceset="CRYSTAL" device="HC49S" package3d_urn="urn:adsk.eagle:package:12071/1"/>
+<part name="IC5" library="memory" library_urn="urn:adsk.eagle:library:279" deviceset="2164" device="" package3d_urn="urn:adsk.eagle:package:19066/1"/>
+<part name="IC6" library="memory" library_urn="urn:adsk.eagle:library:279" deviceset="2164" device="" package3d_urn="urn:adsk.eagle:package:19066/1"/>
+<part name="IC7" library="memory" library_urn="urn:adsk.eagle:library:279" deviceset="2164" device="" package3d_urn="urn:adsk.eagle:package:19066/1"/>
+<part name="IC8" library="memory" library_urn="urn:adsk.eagle:library:279" deviceset="2164" device="" package3d_urn="urn:adsk.eagle:package:19066/1"/>
+<part name="IC9" library="memory" library_urn="urn:adsk.eagle:library:279" deviceset="2164" device="" package3d_urn="urn:adsk.eagle:package:19066/1"/>
+<part name="IC10" library="memory" library_urn="urn:adsk.eagle:library:279" deviceset="2164" device="" package3d_urn="urn:adsk.eagle:package:19066/1"/>
+<part name="IC11" library="memory" library_urn="urn:adsk.eagle:library:279" deviceset="2164" device="" package3d_urn="urn:adsk.eagle:package:19066/1"/>
+<part name="IC12" library="memory" library_urn="urn:adsk.eagle:library:279" deviceset="2164" device="" package3d_urn="urn:adsk.eagle:package:19066/1"/>
 </parts>
 <sheets>
@@
 <instance part="R1" gate="G$1" x="-187.96" y="53.34"/>
 <instance part="Q1" gate="G$1" x="-127" y="58.42" rot="R90"/>
+<instance part="IC5" gate="A" x="-81.28" y="12.7"/>
+<instance part="IC6" gate="A" x="-81.28" y="-30.48"/>
+<instance part="IC7" gate="A" x="-81.28" y="-76.2"/>
+<instance part="IC8" gate="A" x="-81.28" y="-119.38"/>
+<instance part="IC9" gate="A" x="-40.64" y="12.7"/>
+<instance part="IC10" gate="A" x="-40.64" y="-30.48"/>
+<instance part="IC11" gate="A" x="-40.64" y="-76.2"/>
+<instance part="IC12" gate="A" x="-40.64" y="-119.38"/>
 </instances>
 <busses>
@@
 <segment>
 <pinref part="IC2" gate="A" pin="I0"/>
-<wire x1="-12.7" y1="88.9" x2="-55.88" y2="88.9" width="0.1524" layer="91"/>
+<wire x1="-12.7" y1="88.9" x2="-40.64" y2="88.9" width="0.1524" layer="91"/>
 <label x="-53.34" y="88.9" size="1.778" layer="95"/>
 <pinref part="IC3" gate="B" pin="Q"/>
+<wire x1="-40.64" y1="88.9" x2="-55.88" y2="88.9" width="0.1524" layer="91"/>
 <wire x1="-55.88" y1="88.9" x2="-55.88" y2="63.5" width="0.1524" layer="91"/>
 <wire x1="-55.88" y1="63.5" x2="-68.58" y2="63.5" width="0.1524" layer="91"/>
+<wire x1="-40.64" y1="88.9" x2="-40.64" y2="35.56" width="0.1524" layer="91"/>
+<junction x="-40.64" y="88.9"/>
+<wire x1="-40.64" y1="35.56" x2="-58.42" y2="35.56" width="0.1524" layer="91"/>
+<wire x1="-58.42" y1="35.56" x2="-58.42" y2="2.54" width="0.1524" layer="91"/>
+<pinref part="IC9" gate="A" pin="!RAS"/>
+<wire x1="-58.42" y1="2.54" x2="-53.34" y2="2.54" width="0.1524" layer="91"/>
+<pinref part="IC5" gate="A" pin="!RAS"/>
+<wire x1="-93.98" y1="2.54" x2="-99.06" y2="2.54" width="0.1524" layer="91"/>
+<wire x1="-99.06" y1="2.54" x2="-99.06" y2="35.56" width="0.1524" layer="91"/>
+<wire x1="-99.06" y1="35.56" x2="-58.42" y2="35.56" width="0.1524" layer="91"/>
+<junction x="-58.42" y="35.56"/>
+<pinref part="IC10" gate="A" pin="!RAS"/>
+<wire x1="-58.42" y1="2.54" x2="-58.42" y2="-40.64" width="0.1524" layer="91"/>
+<wire x1="-58.42" y1="-40.64" x2="-53.34" y2="-40.64" width="0.1524" layer="91"/>
+<junction x="-58.42" y="2.54"/>
+<pinref part="IC6" gate="A" pin="!RAS"/>
+<wire x1="-99.06" y1="2.54" x2="-99.06" y2="-40.64" width="0.1524" layer="91"/>
+<wire x1="-99.06" y1="-40.64" x2="-93.98" y2="-40.64" width="0.1524" layer="91"/>
+<junction x="-99.06" y="2.54"/>
+<pinref part="IC7" gate="A" pin="!RAS"/>
+<wire x1="-99.06" y1="-40.64" x2="-99.06" y2="-86.36" width="0.1524" layer="91"/>
+<wire x1="-99.06" y1="-86.36" x2="-93.98" y2="-86.36" width="0.1524" layer="91"/>
+<junction x="-99.06" y="-40.64"/>
+<pinref part="IC11" gate="A" pin="!RAS"/>
+<wire x1="-58.42" y1="-40.64" x2="-58.42" y2="-86.36" width="0.1524" layer="91"/>
+<wire x1="-58.42" y1="-86.36" x2="-53.34" y2="-86.36" width="0.1524" layer="91"/>
+<junction x="-58.42" y="-40.64"/>
+<pinref part="IC8" gate="A" pin="!RAS"/>
+<wire x1="-99.06" y1="-86.36" x2="-99.06" y2="-129.54" width="0.1524" layer="91"/>
+<wire x1="-99.06" y1="-129.54" x2="-93.98" y2="-129.54" width="0.1524" layer="91"/>
+<junction x="-99.06" y="-86.36"/>
+<pinref part="IC12" gate="A" pin="!RAS"/>
+<wire x1="-58.42" y1="-86.36" x2="-58.42" y2="-129.54" width="0.1524" layer="91"/>
+<wire x1="-58.42" y1="-129.54" x2="-53.34" y2="-129.54" width="0.1524" layer="91"/>
+<junction x="-58.42" y="-86.36"/>
 </segment>
 </net>

Commit message: resistor
Parts:
- R1: value (none) -> 510
Changed lines of the file:
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@@
 <part name="IC3" library="74xx-us" library_urn="urn:adsk.eagle:library:88" deviceset="74*74" device="N" package3d_urn="urn:adsk.eagle:package:2921/1" technology="LS"/>
 <part name="IC4" library="74xx-us" library_urn="urn:adsk.eagle:library:88" deviceset="74*04" device="N" package3d_urn="urn:adsk.eagle:package:2921/1" technology="LS"/>
-<part name="R1" library="resistor" library_urn="urn:adsk.eagle:library:348" deviceset="R-US_" device="0207/10" package3d_urn="urn:adsk.eagle:package:25939/1"/>
+<part name="R1" library="resistor" library_urn="urn:adsk.eagle:library:348" deviceset="R-US_" device="0207/10" package3d_urn="urn:adsk.eagle:package:25939/1" value="510"/>
 <part name="Q1" library="crystal" library_urn="urn:adsk.eagle:library:204" deviceset="CRYSTAL" device="HC49S" package3d_urn="urn:adsk.eagle:package:12071/1"/>
 <part name="IC5" library="memory" library_urn="urn:adsk.eagle:library:279" deviceset="2164" device="" package3d_urn="urn:adsk.eagle:package:19066/1"/>
