File: eagle/zxclone/board.sch (EAGLE design)
At the start: 14 parts, among them IC2 74LS86N, IC3 74LS74N, IC4 74LS04N

Commit message: govno
Parts:
- added IC13, IC14: (no value), memory:2764
Connections:
- new net B$1: IC1.A0, IC1.A1, IC1.A10, IC1.A11, IC1.A12, IC1.A13, IC1.A14, IC1.A15, IC1.A2, IC1.A3, IC1.A4, IC1.A5, IC1.A6, IC1.A7, IC1.A8, IC1.A9
- new net B$2: IC1.D0, IC1.D1, IC1.D2, IC1.D3, IC1.D4, IC1.D5, IC1.D6, IC1.D7
Other:
- moved on the sheet: IC1
Changed lines of the file:
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@@
 <part name="IC11" library="memory" library_urn="urn:adsk.eagle:library:279" deviceset="2164" device="" package3d_urn="urn:adsk.eagle:package:19066/1"/>
 <part name="IC12" library="memory" library_urn="urn:adsk.eagle:library:279" deviceset="2164" device="" package3d_urn="urn:adsk.eagle:package:19066/1"/>
+<part name="IC13" library="memory" library_urn="urn:adsk.eagle:library:279" deviceset="2764" device="" package3d_urn="urn:adsk.eagle:package:19070/1"/>
+<part name="IC14" library="memory" library_urn="urn:adsk.eagle:library:279" deviceset="2764" device="" package3d_urn="urn:adsk.eagle:package:19070/1"/>
 </parts>
 <sheets>
@@
 </plain>
 <instances>
-<instance part="IC1" gate="1" x="76.2" y="45.72"/>
+<instance part="IC1" gate="1" x="73.66" y="45.72"/>
 <instance part="IC2" gate="A" x="0" y="86.36"/>
 <instance part="IC2" gate="B" x="0" y="66.04"/>
@@
 <instance part="IC11" gate="A" x="-40.64" y="-76.2"/>
 <instance part="IC12" gate="A" x="-40.64" y="-119.38"/>
+<instance part="IC13" gate="A" x="149.86" y="53.34"/>
+<instance part="IC14" gate="A" x="149.86" y="-7.62"/>
 </instances>
 <busses>
@@
 <wire x1="33.02" y1="66.04" x2="33.02" y2="22.86" width="0.1524" layer="91"/>
 <pinref part="IC1" gate="1" pin="CLK"/>
-<wire x1="33.02" y1="22.86" x2="58.42" y2="22.86" width="0.1524" layer="91"/>
+<wire x1="33.02" y1="22.86" x2="55.88" y2="22.86" width="0.1524" layer="91"/>
 </segment>
 </net>
@@
 </segment>
 </net>
+<net name="B$1" class="0">
+<segment>
+<pinref part="IC1" gate="1" pin="A0"/>
+<wire x1="91.44" y1="73.66" x2="101.6" y2="73.66" width="0.1524" layer="91"/>
+</segment>
+<segment>
+<pinref part="IC1" gate="1" pin="A1"/>
+<wire x1="91.44" y1="71.12" x2="101.6" y2="71.12" width="0.1524" layer="91"/>
+</segment>
+<segment>
+<pinref part="IC1" gate="1" pin="A2"/>
+<wire x1="91.44" y1="68.58" x2="101.6" y2="68.58" width="0.1524" layer="91"/>
+</segment>
+<segment>
+<pinref part="IC1" gate="1" pin="A3"/>
+<wire x1="91.44" y1="66.04" x2="101.6" y2="66.04" width="0.1524" layer="91"/>
+</segment>
+<segment>
+<pinref part="IC1" gate="1" pin="A4"/>
+<wire x1="91.44" y1="63.5" x2="101.6" y2="63.5" width="0.1524" layer="91"/>
+</segment>
+<segment>
+<pinref part="IC1" gate="1" pin="A5"/>
+<wire x1="91.44" y1="60.96" x2="101.6" y2="60.96" width="0.1524" layer="91"/>
+</segment>
+<segment>
+<pinref part="IC1" gate="1" pin="A6"/>
+<wire x1="91.44" y1="58.42" x2="101.6" y2="58.42" width="0.1524" layer="91"/>
+</segment>
+<segment>
+<pinref part="IC1" gate="1" pin="A7"/>
+<wire x1="91.44" y1="55.88" x2="101.6" y2="55.88" width="0.1524" layer="91"/>
+</segment>
+<segment>
+<pinref part="IC1" gate="1" pin="A8"/>
+<wire x1="91.44" y1="53.34" x2="101.6" y2="53.34" width="0.1524" layer="91"/>
+</segment>
+<segment>
+<pinref part="IC1" gate="1" pin="A9"/>
+<wire x1="91.44" y1="50.8" x2="101.6" y2="50.8" width="0.1524" layer="91"/>
+</segment>
+<segment>
+<pinref part="IC1" gate="1" pin="A10"/>
+<wire x1="91.44" y1="48.26" x2="101.6" y2="48.26" width="0.1524" layer="91"/>
+</segment>
+<segment>
+<pinref part="IC1" gate="1" pin="A11"/>
+<wire x1="91.44" y1="45.72" x2="101.6" y2="45.72" width="0.1524" layer="91"/>
+</segment>
+<segment>
+<pinref part="IC1" gate="1" pin="A12"/>
+<wire x1="91.44" y1="43.18" x2="101.6" y2="43.18" width="0.1524" layer="91"/>
+</segment>
+<segment>
+<pinref part="IC1" gate="1" pin="A13"/>
+<wire x1="91.44" y1="40.64" x2="101.6" y2="40.64" width="0.1524" layer="91"/>
+</segment>
+<segment>
+<pinref part="IC1" gate="1" pin="A14"/>
+<wire x1="91.44" y1="38.1" x2="101.6" y2="38.1" width="0.1524" layer="91"/>
+</segment>
+<segment>
+<pinref part="IC1" gate="1" pin="A15"/>
+<wire x1="91.44" y1="35.56" x2="101.6" y2="35.56" width="0.1524" layer="91"/>
+</segment>
+</net>
+<net name="B$2" class="0">
+<segment>
+<pinref part="IC1" gate="1" pin="D0"/>
+<wire x1="91.44" y1="30.48" x2="101.6" y2="30.48" width="0.1524" layer="91"/>
+</segment>
+<segment>
+<pinref part="IC1" gate="1" pin="D1"/>
+<wire x1="91.44" y1="27.94" x2="101.6" y2="27.94" width="0.1524" layer="91"/>
+</segment>
+<segment>
+<pinref part="IC1" gate="1" pin="D2"/>
+<wire x1="91.44" y1="25.4" x2="101.6" y2="25.4" width="0.1524" layer="91"/>
+</segment>
+<segment>
+<pinref part="IC1" gate="1" pin="D3"/>
+<wire x1="91.44" y1="22.86" x2="101.6" y2="22.86" width="0.1524" layer="91"/>
+</segment>
+<segment>
+<pinref part="IC1" gate="1" pin="D4"/>
+<wire x1="91.44" y1="20.32" x2="101.6" y2="20.32" width="0.1524" layer="91"/>
+</segment>
+<segment>
+<pinref part="IC1" gate="1" pin="D5"/>
+<wire x1="91.44" y1="17.78" x2="101.6" y2="17.78" width="0.1524" layer="91"/>
+</segment>
+<segment>
+<pinref part="IC1" gate="1" pin="D6"/>
+<wire x1="91.44" y1="15.24" x2="101.6" y2="15.24" width="0.1524" layer="91"/>
+</segment>
+<segment>
+<pinref part="IC1" gate="1" pin="D7"/>
+<wire x1="91.44" y1="12.7" x2="101.6" y2="12.7" width="0.1524" layer="91"/>
+</segment>
+</net>

Commit message: kek
Parts:
- added CENTER, LEFT, RIGHT: 74LS153N, 74xx-us:74LS153N
- added IC15, IC17: 74LS151N, 74xx-us:74LS151N
Connections:
- removed net B$1: IC1.A0, IC1.A1, IC1.A10, IC1.A11, IC1.A12, IC1.A13, IC1.A14, IC1.A15, IC1.A2, IC1.A3, IC1.A4, IC1.A5, IC1.A6, IC1.A7, IC1.A8, IC1.A9
- removed net B$2: IC1.D0, IC1.D1, IC1.D2, IC1.D3, IC1.D4, IC1.D5, IC1.D6, IC1.D7
- new net A0: IC1.A0, IC13A.A0, IC14A.A0
- new net A1: IC1.A1, IC13A.A1, IC14A.A1
- new net A10: IC1.A10, IC13A.A10, IC14A.A10
- new net A11: IC1.A11, IC13A.A11, IC14A.A11
- new net A12: IC1.A12, IC13A.A12, IC14A.A12
- new net A13: IC1.A13
- new net A14: IC1.A14
- new net A15: IC1.A15
- new net A2: IC1.A2, IC13A.A2, IC14A.A2
- new net A3: IC1.A3, IC13A.A3, IC14A.A3
- new net A4: IC1.A4, IC13A.A4, IC14A.A4
- new net A5: IC1.A5, IC13A.A5, IC14A.A5
- new net A6: IC1.A6, IC13A.A6, IC14A.A6
- new net A7: IC1.A7, IC13A.A7, IC14A.A7
- new net A8: IC1.A8, IC13A.A8, IC14A.A8
- new net A9: IC1.A9, IC13A.A9, IC14A.A9
- new net D0: IC1.D0, IC13A.O0, IC14A.O0, IC5.DI
- new net D1: IC1.D1, IC13A.O1, IC14A.O1, IC9.DI
- new net D2: IC1.D2, IC13A.O2, IC14A.O2, IC6.DI
- new net D3: IC1.D3, IC10.DI, IC13A.O3, IC14A.O3
- new net D4: IC1.D4, IC13A.O4, IC14A.O4, IC7.DI
- new net D5: IC1.D5, IC11.DI, IC13A.O5, IC14A.O5
- new net D6: IC1.D6, IC13A.O6, IC14A.O6, IC8.DI
- new net D7: IC1.D7, IC12.DI, IC13A.O7, IC14A.O7
- new net N$10: CENTERA.1Y, IC5.A1
- new net N$11: IC17A.W, IC5.A2
- new net N$12: IC5.A3, LEFTA.1Y
- new net N$13: CENTERA.2Y, IC5.A4
- new net N$14: IC5.A5, RIGHTA.2Y
- new net N$15: IC5.A6, LEFTA.2Y
- new net N$16: IC5.A7, RIGHTA.1Y
- new net N$9: IC15A.W, IC5.A0
Other:
- moved on the sheet: IC1, IC10, IC11, IC12, IC13, IC14, IC5, IC6, IC7, IC8, IC9
