File: eagle/zxclone/board.sch (EAGLE design)
At the start: 23 parts, among them IC15 74LS174N, IC16 74LS02N, IC2 74LS86N, IC3 74LS74N, IC4 74LS04N

Commit message: tajk
Parts:
- added IC17: 74LS04N, 74xx-us:74LS04N
- added IC18: 74S260N, 74xx-us:74S260N
- added IC19: 74LS32N, 74xx-us:74LS32N
- added R2, R3, R4, R5, R6, R7, R8: (no value), resistor:R-US_0207/10
- added V1, V2, V3: 74193N, 74ttl-din:74193N
Connections:
- new net N$10: CENTER2A.B, LEFT2A.B, RIGHT2A.B
- new net N$11: LEFT2A.1C3, R2.2, V11.QA
- new net N$12: R2.1, R3.2
- new net N$13: LEFT2A.1C2, R4.2
- new net N$14: R4.1, R5.2
- new net N$15: R5.1, R6.2
- new net N$16: R6.1, R7.2
- new net N$17: IC17A.O, R7.1
- new net N$18: LEFT2A.2C2, V11.QB
- new net N$19: CENTER2A.2C3, IC18A.I1, LEFT2A.2C3, RIGHT2A.2C3
- new net N$20: IC1.INT, IC17B.O
- new net N$21: CENTER2A.1C3, R8.2
- new net N$22: IC17F.O, R8.1
- new net N$23: CENTER2A.1C2, V21.QB
- new net N$24: IC19B.O, RIGHT2A.1C3
- new net N$25: RIGHT2A.1C2, V21.QC
- new net N$26: CENTER2A.2C2, V31.QD
- new net N$27: RIGHT2A.2C2, V21.QD
- new net N$28: LEFT7A.D3, V31.QB
- new net TOINTELPIN13: R3.1
- net GND: now also CENTER2A.1G, CENTER2A.2G, LEFT2A.1G, LEFT2A.2G, RIGHT2A.1G, RIGHT2A.2G
- net N$3: now also CENTER2A.A, LEFT2A.A, RIGHT2A.A
