File: eagle/zxclone/boardv2.sch (EAGLE design)
At the start: 21 parts, among them IC1 74AS04N, IC10 74LS02N, IC11 74LS86N, IC12 74LS00N, IC13 74LS366N, IC14 7432N, IC2 74LS74N, IC3 74LS192N, IC4 74LS192N, IC5 74LS192N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

Commit message: build
Parts:
- added IC15, IC16: 74S151N, 74xx-us:74S151N
- added IC17, IC18, IC19: 74LS153N, 74xx-us:74LS153N
- added IC20: (no value), zilog:Z80CPU
- added IC21, IC22, IC23, IC24, IC25, IC26, IC27, IC28: (no value), memory:2164
- added IC29: (no value), memory:2764
Connections:
- new net A0: IC20.A0, IC29A.A0
- new net A1: IC20.A1, IC29A.A1
- new net A10: IC20.A10, IC29A.A10
- new net A11: IC20.A11, IC29A.A11
- new net A12: IC20.A12, IC29A.A12
- new net A13: IC20.A13
- new net A14: IC20.A14
- new net A15: IC20.A15
- new net A2: IC20.A2, IC29A.A2
- new net A3: IC20.A3, IC29A.A3
- new net A4: IC20.A4, IC29A.A4
- new net A5: IC20.A5, IC29A.A5
- new net A6: IC20.A6, IC29A.A6
- new net A7: IC20.A7, IC29A.A7
- new net A8: IC20.A8, IC29A.A8
- new net A9: IC20.A9, IC29A.A9
- new net D0: IC20.D0, IC29A.O0
- new net D1: IC20.D1, IC29A.O1
- new net D2: IC20.D2, IC29A.O2
- new net D3: IC20.D3, IC29A.O3
- new net D4: IC20.D4, IC29A.O4
- new net D5: IC20.D5, IC29A.O5
- new net D6: IC20.D6, IC29A.O6
- new net D7: IC20.D7, IC29A.O7
